File: f1/pcb/sc02_drive.kicad_sch (KiCad schematic)
At the start: 84 parts, among them J1 BAT 3S, J10 LICHTEN, J2 MOTOR 1, J3 MOTOR 2, J4 SERVO, J5 HALL, J6 ZONNEPANEEL, J7 I2C, J8 USB-C, J9 PI 4, Q1 AOD4185, Q2 2N7002, Q3 2N7002, Q4 AO3400A, SW1 RESET, SW2 BOOT, U1 TPS54560B, U10 USBLC6-2SC6, U2 AMS1117-3.3, U3 ESP32-S3-WROOM-1-N16R8, U4 DRV8871, U5 DRV8871, U6 INA226

Commit message: SC-02 floor board v2: the whole floor is the PCB (XT60, fuse, ELRS RP2 pads, Pi UART, USB-C at the edge); body gets a USB-C opening
Co-Authored-By: Claude Opus 5.5 <noreply@anthropic.com>
Parts:
- removed Q2, Q3: 2N7002, sc02:SOT-23, symbol sc02:2N7002
- removed R14, R15: 100k, sc02:R_0603_1608Metric, symbol sc02:R
- added F1: 10A, sc02:R_2512_6332Metric, symbol sc02:Fuse
- added H10, H11, H12, H13, H14, H18, H19, H20, H21, H22, H23, H24, H25, H26, H27, H28, H29, H30, H31, H5, H6, H7, H8, H9: 3.2, sc02:Hole_3.2mm, symbol sc02:MountingHole
- added H15, H16, H17: 2.6, sc02:Hole_2.6mm, symbol sc02:MountingHole
- added H32: 6.2, sc02:Hole_6.2mm, symbol sc02:MountingHole
- added J11: SCHAKELAAR, sc02:SolderWire_2pad_P5mm_SW, symbol sc02:Conn_01x02
- added J12: ELRS RP2, sc02:Pads_ELRS_RX, symbol sc02:Conn_01x04
- added J13: 5V PI, sc02:SolderWire_2pad_P5mm_5V, symbol sc02:Conn_01x02
- added R29, R30: 100, sc02:R_0603_1608Metric, symbol sc02:R
- H1, H2, H3, H4: value M2.5 -> 3.2; footprint sc02:MountingHole_2.75mm_M2.5_Pi -> sc02:Hole_3.2mm
- J1: value BAT 3S -> XT60; footprint sc02:SolderWire_2pad_P7mm_D2.2mm_BAT -> sc02:AMASS_XT60-M_1x02_P7.20mm_Vertical; MPN solder pads for the XT60 lead (14-16 AWG) -> AMASS XT60-M (male, vertical): the LiPo plugs in from above
- J8: MPN HRO TYPE-C-31-M-12 -> HRO TYPE-C-31-M-12 (at the floor edge: reachable through th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
- J9: value PI 4 -> PI UART; footprint sc02:PinSocket_2x20_P2.54mm_Vertical -> sc02:Pads_PI_UART; symbol sc02:Conn_02x20_Odd_Even -> sc02:Conn_01x03; MPN 2x20 socket 2.54 mm, 8.5 mm (on the bottom side, onto the P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 -> solder pads: wires to the Pi 4 header (pin 6 GND, pin 8 TXD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
- SW2: MPN CK KMR221G (4.2x2.8 tact) - also race-mode button -> CK KMR221G (4.2x2.8 tact) - also the race-mode button
Connections:
- net GND: now also J9.1 (Pin_1), J12.1 (Pin_1), J13.1 (Pin_1); no longer J9.14 (Pin_14), J9.20 (Pin_20), J9.25 (Pin_25), J9.30 (Pin_30), J9.34 (Pin_34), J9.39 (Pin_39), J9.6 (Pin_6), J9.9 (Pin_9)
- net HALL: now also U3.31 (IO38); no longer U3.18 (IO10)
- net PI_RXD: now also J9.3 (Pin_3); no longer J9.10 (Pin_10)
- net PI_TXD: now also J9.2 (Pin_2); no longer J9.8 (Pin_8)
- net V5: now also J12.2 (Pin_2), J13.2 (Pin_2); no longer J9.2 (Pin_2), J9.4 (Pin_4)
- net VBAT_RAW: now also J11.2 (Pin_2); no longer J1.2 (Pin_2)
- net ELRS_TX: now reaches U3.8 (IO15)
- net ELRS_TX: now also R30.1
- net ELRS_RX: now reaches U3.9 (IO16)
- net ELRS_RX: now also R29.2
- removed net PI_ESP_BOOT: J9.11 (Pin_11)
- removed net PI_ESP_EN: J9.7 (Pin_7)
- new net BAT_F: F1.2, J11.1 (Pin_1)
- new net BAT_IN: F1.1, J1.2 (Pin_2)
- new net ELRS_RX_IN: J12.3 (Pin_3), R29.1
- new net ELRS_TX_OUT: J12.4 (Pin_4), R30.2
- no-connect marks 49 -> 21
Other:
- note added: "BATTERIJ 3S: XT60, ZEKERING, SCHAKELAAR, STROOMMETING"
- note added: "BEVESTIGING (VLOERGATEN)"
- note added: "Battery: XT60 -> 10 A fuse -> power switch (pads, switch in the floor hole) -> P-MOSFET reverse protection -> 2 mOhm shunt (INA226 0x40) -> VBUS: motors + buck."
- note added: "ELRS-ONTVANGER + PI UART"
- note added: "Motors: DRV8871 IN1/IN2 (M1: IO4/IO5, M2: IO6/IO7), current limit 64 / 18k = 3.55 A. Servo IO9 (100 R), hall A3144 IO38 (10k pull-up), lights IO11 (AO3400A), panel ADC IO8 (100k/33k)."
- note added: "Pi 4: UART pads (ESP IO17 TX / IO18 RX via 1k) to Pi pins 8/10 + 5V PI pads (pin 2/4 + 6). USB-C at the floor edge (body opening) for flashing. ELRS receiver (RadioMaster RP2, CRSF 420k) on IO15 TX / IO16 RX."
- note added: "SC-02 FLOOR BOARD v2.0 - the whole car floor is this PCB (2 mm, 4 layers): ESP32-S3 + 2x DRV8871 + INA226 + 5 V 5 A buck (generated by tools/build_sch.py from tools/design.py)"
- note added: "USB-C (FLASHEN / DEBUG VAN BUITENAF)"
- note removed: "BATTERIJ 3S + STROOMMETING"
- note removed: "BEVESTIGING"
- note removed: "Battery 3S LiPo (9-12.6 V) -> P-MOSFET reverse protection -> 2 mOhm shunt (INA226 @ 0x40, I2C IO1/IO2) -> VBUS: motors + buck. Buck 5 V -> Pi 4 header pins 2/4, servo, hall, lights."
- note removed: "Motors: DRV8871 IN1/IN2 (M1: IO4/IO5, M2: IO6/IO7), current limit 64 / 18k = 3.55 A. Servo IO9 (100 R), hall A3144 IO10 (10k pull-up to 3V3), lights IO11 (AO3400A low side), panel ADC IO8 (100k/33k)."
- note removed: "Pi link: ESP IO17 (TX) -> 1k -> Pi GPIO15 RXD (pin 10), Pi GPIO14 TXD (pin 8) -> 1k -> ESP IO18 (RX). Pi GPIO4 (pin 7) resets the ESP, Pi GPIO17 (pin 11) holds BOOT: flash it from the Pi with esptool."
- note removed: "RASPBERRY PI 4 (40-PIN)"
- note removed: "SC-02 DRIVE BOARD v1.0 - ESP32-S3 + 2x DRV8871 + INA226 + 5 V 5 A buck, sits on the Raspberry Pi 4 like a HAT (generated by tools/build_sch.py from tools/design.py)"
- note removed: "The 40-pin socket sits on the BOTTOM side. Do not power the Pi from its own USB-C at the same time (the board feeds its 5 V pins directly)."
- note removed: "USB-C ESP32"
- title: SC-02 drive board -> SC-02 floor board
- moved on the sheet: C1, C14, C15, C16, C17, C18, C19, C20, C21, C22, C23, C29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

Commit message: SC-02 drive board v3: compact board on standoffs, no Pi, built-in ExpressLRS receiver (ESP32-C3 + E28 SX1280, Generic C3 2400), JST-XH solar connector
Co-Authored-By: Claude Opus 5.5 <noreply@anthropic.com>
Parts:
- removed H10, H11, H12, H13, H14, H18, H19, H20, H21, H22, H23, H24, H25, H26, H27, H28, H29, H30, H31, H5, H6, H7, H8, H9: 3.2, sc02:Hole_3.2mm, symbol sc02:MountingHole
- removed H15, H16, H17: 2.6, sc02:Hole_2.6mm, symbol sc02:MountingHole
- removed H32: 6.2, sc02:Hole_6.2mm, symbol sc02:MountingHole
- removed J13: 5V PI, sc02:SolderWire_2pad_P5mm_5V, symbol sc02:Conn_01x02
- removed J9: PI UART, sc02:Pads_PI_UART, symbol sc02:Conn_01x03
- removed R16, R17: 1k, sc02:R_0603_1608Metric, symbol sc02:R
- added C30, C33: 10u, sc02:C_0805_2012Metric, symbol sc02:C
- added C31: 22u, sc02:C_0805_2012Metric, symbol sc02:C
- added C32, C34: 100n, sc02:C_0603_1608Metric, symbol sc02:C
- added C35: 1u, sc02:C_0603_1608Metric, symbol sc02:C
- added D10: SK6812MINI-E, sc02:LED-SMD_4P-L3.2-W2.8-LS5.9_SK6812MINI-E, symbol sc02:SK6812MINI-E
- added D9: SS14, sc02:D_SMA, symbol sc02:SS14
- added JP1: ZON>5V, sc02:SolderJumper-2_P1.3mm_Open_RoundedPad1.0x1.5mm, symbol sc02:SolderJumper_2_Open
- added R31, R32, R33: 10k, sc02:R_0603_1608Metric, symbol sc02:R
- added R34, R35: 1k, sc02:R_0603_1608Metric, symbol sc02:R
- added SW3: BIND, sc02:SW_Push_1P1T_NO_CK_KMR2, symbol sc02:SW_Push
- added U11: ESP32-C3-MINI-1-N4, sc02:WIFIM-SMD_ESP32-C3-MINI-1, symbol sc02:ESP32-C3-MINI-1
- added U12: E28-2G4M12S, sc02:WIRELM-SMD_E28-2G4M12S, symbol sc02:E28-2G4M12S
- added U13: AMS1117-3.3, sc02:SOT-223-3_TabPin2, symbol sc02:AMS1117-3.3
- H1, H2, H3, H4: value 3.2 -> M3
- J12: value ELRS RP2 -> RX USB; footprint sc02:Pads_ELRS_RX -> sc02:Pads_RX_USB; symbol sc02:Conn_01x04 -> sc02:Conn_01x03; MPN solder pads for a RadioMaster RP2 ELRS receiver (stick it o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 -> test pads: USB D-/D+/GND of the receiver C3 (first flash)
- J6: footprint sc02:SolderWire_2pad_P4mm_S -> sc02:JST_XH_B2B-XH-A_1x02_P2.50mm_Vertical; MPN solder pads, solar panel 5 V (measured only) -> JST XH 2-pin (B2B-XH-A): plug the solar panel in (5 V 1 W)
- J8: MPN HRO TYPE-C-31-M-12 (at the floor edge: reachable through th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 -> HRO TYPE-C-31-M-12 (board edge)
Connections:
- net GND: now also J12.3 (Pin_3), C30.2, C31.2, C32.2, C33.2, C34.2, C35.2, D10.1 (GND), SW3.2, U11.1 (GND), U11.11 (GND), U11.14 (GND), U11.2 (GND), U11.36 (GND), U11.37 (GND), U11.38 (GND), U11.39 (GND), U11.40 (GND), U11.41 (GND), U11.42 (GND), U11.43 (GND), U11.44 (GND), U11.45 (GND), U11.46 (GND), U11.47 (GND), U11.48 (GND), U11.49 (GND), U11.50 (GND), U11.51 (GND), U11.52 (GND), U11.53 (GND), U12.14 (GND), U12.2 (GND), U12.7 (GND), U12.8 (GND), U13.1 (GND); no longer J12.1 (Pin_1)
- net PANEL: now also D9.2 (A)
- net V5: now also C30.1, JP1.2 (B), U13.3 (VI); no longer J12.2 (Pin_2)
- net ELRS_RX_IN renamed RX_SERIAL_OUT
- net RX_SERIAL_OUT: now also U11.31 (TXD0); no longer J12.3 (Pin_3)
- net ELRS_TX_OUT renamed RX_SERIAL_IN
- net RX_SERIAL_IN: now also U11.30 (RXD0); no longer J12.4 (Pin_4)
- net ESP_RX renamed RX_BOOT_CTL
- net RX_BOOT_CTL: now also R35.1
- net ESP_TX renamed RX_EN_CTL
- net RX_EN_CTL: now also R34.1
- new net 3V3_RX: C31.1, C32.1, C33.1, C34.1, D10.3 (VDD), R31.1, R32.1, R33.1, U11.3 (3V3), U12.1 (VCC), U13.2 (VO)
- new net PANEL_D: D9.1 (K), JP1.1 (A)
- new net RF_BUSY: U11.6 (IO3), U12.10 (BUSY)
- new net RF_DIO1: U11.13 (IO1), U12.11 (DIO1)
- new net RF_MISO: U11.19 (IO5), U12.3 (MISO_TX)
- new net RF_MOSI: U11.18 (IO4), U12.4 (MOSI_RX)
- new net RF_NSS: U11.21 (IO7), U12.6 (NSS_CTS)
- new net RF_RST: U11.5 (IO2), U12.9 (NRESET)
- new net RF_SCK: U11.20 (IO6), U12.5 (SCK_RTSN)
- new net RX_BOOT: R32.2, R35.2, SW3.1, U11.23 (IO9)
- new net RX_EN: C35.1, R31.2, R34.2, U11.8 (EN)
- new net RX_LED: D10.2 (DIN), R33.2, U11.22 (IO8)
- new net RX_USB_DM: J12.1 (Pin_1), U11.26 (IO18)
- new net RX_USB_DP: J12.2 (Pin_2), U11.27 (IO19)
- no-connect marks 21 -> 40
Other:
- note added: "BEVESTIGING"
- note added: "BUCK 5 V 5 A (ESP32, SERVO, LICHTEN)"
- note added: "Battery: XT60 -> 10 A fuse -> power switch pads -> P-MOSFET reverse protection -> 2 mOhm shunt (INA226 0x40) -> VBUS: motors + buck."
- note added: "ELRS-ONTVANGER (ESP32-C3 + SX1280)"
- note added: "ELRS: ESP32-C3-MINI-1 + E28-2G4M12S (SX1280) wired as ExpressLRS "Generic C3 2400" (SCK 6, MOSI 4, MISO 5, NSS 7, BUSY 3, DIO1 1, RST 2, LED 8, button 9). CRSF: C3 TX21 -> S3 IO16, S3 IO15 -> C3 RX20."
- note added: "Motors: DRV8871 IN1/IN2 (M1: IO4/IO5, M2: IO6/IO7), limit 64/18k = 3.55 A. Servo IO9 (100 R), hall IO38 (10k pull-up), lights IO11 (AO3400A), solar panel JST-XH, ADC IO8 (100k/33k), JP1 = panel -> 5 V."
- note added: "S3 IO17 -> C3 EN (reset), S3 IO18 -> C3 IO9 (bootloader). First flash of the C3: USB pads RX USB (D-, D+, GND) or WiFi. Bind: BIND button (C3 IO9)."
- note added: "SC-02 DRIVE BOARD v3.0 - compact board on M3 standoffs (battery on top): ESP32-S3 + 2x DRV8871 + INA226 + 5 V 5 A buck + built-in ExpressLRS receiver (generated by tools/build_sch.py from tools/design.py)"
- note removed: "BEVESTIGING (VLOERGATEN)"
- note removed: "BUCK 5 V 5 A (PI 4 + SERVO)"
- note removed: "Battery: XT60 -> 10 A fuse -> power switch (pads, switch in the floor hole) -> P-MOSFET reverse protection -> 2 mOhm shunt (INA226 0x40) -> VBUS: motors + buck."
- note removed: "ELRS-ONTVANGER + PI UART"
- note removed: "Motors: DRV8871 IN1/IN2 (M1: IO4/IO5, M2: IO6/IO7), current limit 64 / 18k = 3.55 A. Servo IO9 (100 R), hall A3144 IO38 (10k pull-up), lights IO11 (AO3400A), panel ADC IO8 (100k/33k)."
- note removed: "Pi 4: UART pads (ESP IO17 TX / IO18 RX via 1k) to Pi pins 8/10 + 5V PI pads (pin 2/4 + 6). USB-C at the floor edge (body opening) for flashing. ELRS receiver (RadioMaster RP2, CRSF 420k) on IO15 TX / IO16 RX."
- note removed: "SC-02 FLOOR BOARD v2.0 - the whole car floor is this PCB (2 mm, 4 layers): ESP32-S3 + 2x DRV8871 + INA226 + 5 V 5 A buck (generated by tools/build_sch.py from tools/design.py)"
- moved on the sheet: C17, C18, C19, H1, H2, H3, H4, J10, J7, Q4, R11, R12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

Commit message: Drive board v3: brushless ESC output (IO4) + ESC/motor NTC (IO5) instead of 2x DRV8871
Co-Authored-By: Claude Opus 5.5 <noreply@anthropic.com>
Parts:
- removed C20, C22: 10u 25V, sc02:C_1206_3216Metric, symbol sc02:C
- removed C21, C23: 100n, sc02:C_0603_1608Metric, symbol sc02:C
- removed U4, U5: DRV8871, sc02:Texas_HTSOP-8-1EP_3.9x4.9mm_P1.27mm_EP2.95x4.9mm_Mask2.4x3.1mm_ThermalVias, symbol sc02:DRV8871DDA
- J2: value MOTOR 1 -> ESC; footprint sc02:SolderWire_2pad_P5mm_M -> sc02:PinHeader_1x03_P2.54mm_Vertical; symbol sc02:Conn_01x02 -> sc02:Conn_01x03; MPN solder pads, motor leads -> 1x3 pin header 2.54 (ESC signal lead: black GND, red BEC NO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
- J3: value MOTOR 2 -> ESC TEMP; MPN solder pads, motor leads -> solder pads: 10k NTC glued on the ESC / motor can (temperat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
- R20: value 18k -> 100; MPN 0603 18k 1% -> 0603 100 1%
- R21: value 18k -> 10k; MPN 0603 18k 1% -> 0603 10k 1% (NTC divider)
Connections:
- net M1_A is gone; now on net GND: J2.1 (Pin_1)
- net M1_IN1 is gone; now on net ESC_PWM: U3.4 (IO4)
- net M2_A is gone; now on net GND: J3.1 (Pin_1)
- net M2_B is gone; now on net ESC_NTC: J3.2 (Pin_2)
- net M2_ILIM is gone; now on net ESC_NTC: R21.1
- net 3V3: now also R21.2
- net GND: no longer R20.2, R21.2
- net M1_B: no longer names the net of J2.2 (Pin_2)
- net M1_ILIM renamed ESC_PWM
- net M1_IN2 renamed ESC_NTC
- net M2_IN1: no longer names the net of U3.6 (IO6)
- net M2_IN2: no longer names the net of U3.7 (IO7)
- new net ESC_SIG: J2.3 (Pin_3), R20.2
- no-connect marks 40 -> 43
Other:
- note added: "ESC (BRUSHLESS)"
- note added: "Motor: one brushless 2435 4500KV on a 40 A ESC (battery via Y-cable, not through this board). ESC signal IO4 (100 R), ESC/motor NTC IO5 (10k divider). Servo IO9 (100 R), hall IO38 (10k pull-up), lights IO11 (AO3400A), solar panel JST-XH, ADC IO8 (100k/33k), JP1 = panel -> 5 V."
- note added: "SC-02 DRIVE BOARD v3.0 - compact board on M3 standoffs (battery on top): ESP32-S3 + brushless ESC output + INA226 + 5 V 5 A buck + built-in ExpressLRS receiver (generated by tools/build_sch.py from tools/design.py)"
- note removed: "MOTOR 1 (DRV8871)"
- note removed: "MOTOR 2 (DRV8871)"
- note removed: "Motors: DRV8871 IN1/IN2 (M1: IO4/IO5, M2: IO6/IO7), limit 64/18k = 3.55 A. Servo IO9 (100 R), hall IO38 (10k pull-up), lights IO11 (AO3400A), solar panel JST-XH, ADC IO8 (100k/33k), JP1 = panel -> 5 V."
- note removed: "SC-02 DRIVE BOARD v3.0 - compact board on M3 standoffs (battery on top): ESP32-S3 + 2x DRV8871 + INA226 + 5 V 5 A buck + built-in ExpressLRS receiver (generated by tools/build_sch.py from tools/design.py)"
- moved on the sheet: C14, C15, C16, C17, C18, C19, C29, C30, C31, C32, C33, C34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

Commit message: SC-02 CAD: one 2435 brushless (11T/35T m0.8) on a motor plate + strap, ESC beside the motor, drive PCB v3 on 4 mm posts, 2S LiPo tray above the PCB, acrylic floor; interference pairs 0. PCB: J4 servo lead soldered flat (not fitted)
Co-Authored-By: Claude Opus 5.5 <noreply@anthropic.com>
Parts:
- J4: MPN 1x3 pin header 2.54 (MG90S: brown GND, red 5 V, orange sign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 -> NOT FITTED: solder the MG90S lead straight into the holes, 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; now not fitted
Changed lines of the file:
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@@
 		(in_bom yes)
 		(on_board yes)
-		(dnp no)
+		(dnp yes)
 		(property "Reference" "J4"
 			(at 226.06 29.25 0)
@@
 			)
 		)
-		(property "MPN" "1x3 pin header 2.54 (MG90S: brown GND, red 5 V, orange signal)"
+		(property "MPN" "NOT FITTED: solder the MG90S lead straight into the holes, flat (battery tray sits 8 mm above). Brown GND, red 5 V, orange signal"
 			(at 226.06 35.56 0)
 			(effects

Commit message: Renders: real KiCad drive PCB (matte black) + real 2S LiPo with label, leads, XT60 and balance plug; name Kobe Vanrobaeys
Co-Authored-By: Claude Opus 5.5 <noreply@anthropic.com>
Other:
- company: Kobe Van Robaeys -> Kobe Vanrobaeys
Changed lines of the file:
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@@
 		(date "2026-10-18")
 		(rev "2.0")
-		(company "Kobe Van Robaeys")
+		(company "Kobe Vanrobaeys")
 		(comment 1 "drive board v3: ESP32-S3 + ESC output + ELRS + INA226 + buck")
 	)
